Commit message: work!

File: ur5e_robotiq/ur5e_robotiq_description/urdf/ur5e_robotiq.urdf.xacro (robot description, xacro)
@@ -40,5 +40,5 @@
 		<parent link="world"/>
 		<child link="camera_link"/>
-		<origin xyz="0.27 0.9 1.23" rpy="0.0 ${pi/2} 0.0"/>
+		<origin xyz="0.27 0.9 1.5" rpy="${pi/4} ${pi/2} 0"/>
 	  </joint>
 	</xacro:unless>

Commit message: using waypoint

File: ur5e_robotiq/ur5e_robotiq_description/urdf/ur5e_robotiq.urdf.xacro (robot description, xacro)
@@ -7,4 +7,6 @@
   <xacro:include filename="$(find ur_e_description)/urdf/common.gazebo.xacro" />
   <!-- ur5e -->
+  <xacro:property name="damping_value" value="10" />
+  <xacro:property name="friction_value" value="0.1" />
   <xacro:include filename="$(find ur_e_description)/urdf/ur5e.urdf.xacro" />
    <xacro:include filename="$(find robotiq_85_description)/urdf/robotiq_85_gripper.urdf.xacro" />
